File: STM32WB55CG/STM32WB55_QFN48_IPD_REF_BOARD.sch (KiCad schematic (older format))
At the start: 64 parts, among them IC1 ECMF02-2AMX6, J1 USB_B_Micro, U1 STM32WB55CG, U2 MCP1640CCH, U3 ADS1115IDGS, U4 BNO055_my, Y1 NX2520SA-32MHz, Y2 NX2012SA-32768K, Y3 NX2012SA-32768K

Commit message: schema complete
Parts:
- removed C13: 0p8, symbol Device:C_Small
- removed C18: 10n, symbol Device:C_Small
- removed C19: Not fitted, symbol Device:C_Small
- removed C26: 22p, symbol Device:C_Small
- removed C6: 100n, symbol Device:C_Small
- removed C_2: 100p, symbol Device:C_Small
- removed D1: ESDA7P60-1U1M, ESDA7P601U1M, symbol ESDA7p6:ESDA7P60-1U1M
- removed FL1: DEA162450BT-1295A1, DEA162450BT1295A1, symbol BPF:DEA162450BT-1295A1
- removed FSR1, FSR2, FSR3: FSR04, symbol myanalog:FSR04
- removed IC1: ECMF02-2AMX6, SON50P150X170X55-6N-D, symbol ECMUSB:ECMF02-2AMX6
- removed JP2: SolderJumper Open, symbol Jumper:SolderJumper_2_Open
- removed L3: 2n7, symbol Device:L_Small
- removed L4: 3n6, symbol Device:L_Small
- removed R1: 100K, symbol Device:R
- removed R4, R5: 100K, symbol Device:R_Small
- removed U1: STM32WB55CG, symbol ST32WB55CG:STM32WB55CG
- added C11, C16: 1u, symbol Device:C_Small
- added C12: 100n, symbol Device:C_Small
- added C14: 10n, symbol Device:C_Small
- added D1: LED Blue, symbol Device:LED
- added D3: 1N4148WT, Diode_SMD:D_SOD-523, symbol Diode:1N4148WT
- added FB2: MMZ2012Y152BTD25, symbol Device:Ferrite_Bead_Small
- added FB3: MMZ2012Y152BT000, symbol Device:Ferrite_Bead_Small
- added FL1: MLPF-WB55-01E3, 0Pretty:MLPF-WB55-02E3, symbol FilterBT:MLPF-WB55-01E3
- added IC1: LD3985M33R, USBRegulator:SOT95P280X145-5N, symbol UBS5-3V3:LD3985M33R
- added IC2: USBLC6-2SC6, USB_data:SOT95P280X145-6N, symbol USB_svab:USBLC6-2SC6
- added J2: Conn_01x06_Male, symbol Connector:Conn_01x06_Male
- added J3: Conn_01x04_Male, symbol Connector:Conn_01x04_Male
- added J4: Conn_01x05_Male, symbol Connector:Conn_01x05_Male
- added J5: Conn_01x03_Male, symbol Connector:Conn_01x03_Male
- added L3: 10n, symbol Device:L
- added R1: 100K, symbol Device:R_Small
- added R12, R13, R2, R3: 10K, symbol Device:R_Small
- added U2: STM32WB55CG, ST32_3D:STM32WB55CGU7, symbol ST32WB55CG:STM32WB55CG
- added U3: MLL1200S TE, Package_SO:TSSOP-20_4.4x6.5mm_P0.65mm, symbol Analog_Switch:ADG734
- added ed1: RECE.20279.001E.01, RECE_antena_connector:RECE.20279.001E.01, symbol konektorAntennaaRECE:RECE.20279.001E.01
- BT1: footprint (none) -> Battery:BatteryHolder_Keystone_2466_1xAAA
- C15: value 0p3 -> 100n
- C20: value 1p8 = datasheet 1p2 -> 100n
- C21: value 0u1 -> 1u
- C22: value 100n -> 1u
- C23: value 120n -> 1u
- C24: value 1u -> 22p
- J1: footprint (none) -> microUSB:UB-MC5BR3-SDWP604-4S-TF
- JP1: footprint (none) -> Jumper:SolderJumper-2_P1.3mm_Open_TrianglePad1.0x1.5mm
- R6: value 100K -> 10K
- R7, R8: value 100K?????????? -> 100K
- R9: value 10K -> 100K
- Y1: footprint (none) -> Crystal:Crystal_SMD_2520-4Pin_2.5x2.0mm
- Y2, Y3: footprint (none) -> Crystal:Crystal_SMD_2012-2Pin_2.0x1.2mm
- renumbered C2 to C1, C11 to C13, C14 to C17, C16 to C18, C17 to C19, C4 to C2, C5 to C3, C9 to C4, C8 to C5, C12 to C6, C1 to C7, C3 to C8, C7 to C9, R2 to R4, R3 to R5, U2 to U1, U3 to U5
Connections:
- net labels added: 3v3fromBAT, 3v3fromUSB, ADC_ALERT, BNO055_RESET, GENERAL_PIN_OUT1, GENERAL_PIN_OUT2, GENERAL_PIN_OUT3, LED_BLUE, SYS_JTCK-SWCLK, SYS_JTDO-SWO, SYS_JTMS-SWDIO, USB_D+, USB_D-
- net labels removed: BL_IND, B_BOOT_PIN, I2C_ADDR, NRESET, USB_DM, USB_DP, VDD, VDDIO, VLXSMPS, VSSSMPS
- wire segments 229 -> 220
- no-connect marks 21 -> 17
Other:
- note added: "BOOT=0 Default position, connected to GND\nBOOT=1 Connected to 3.3V"
- note added: "Coaxial antenna \nconnector"
- note added: "FSR04 sensor x3"
- note added: "For DEBUGGING ONLY\nThese pins are not necessary \njust in case MCU comes without \nDFU firmware (allows USB programming)\n3.3V and GND are in Analog section"
- note added: "LED for debugging purposes"
- note added: "Oscilator section 32MHz and 32768 kHz crystals\nBoot pin for loading booloader and NReset pin"
- note added: "Pin setup for USB and peripherals"
- note added: "Pinout section"
- note added: "Power section"
- note added: "Power selector switch"
- note added: "Reference design from datasheet for MCP1640 step-up from 1.5V battery to 3.3V"
- note added: "SMPS and RF section"
- note added: "SMPS is not necessary but makes MCU, \nespecially Bluetooth connection, \nmore efficient and less power hungry"
- note added: "ST-Link"
- note added: "STM32WB microcontroller section"
- note added: "SpyPen \nThis pen uses ST32WB55 wireless Bluetooth LE microcontroller. \nPowered by a 1.5 AAAA or AAA battery thanks to MCP1640 stepup to 3.3V\nI2C connections to peripherals:\n1. TI ADS1115 for converting analog FSR04 force input to digital \n2. Bosch BNO055 for 9-way motion detection - Accelerometer, Gyroscope, Magnetometer\n\nThis is a prototype. It has few unnecessary parts \n(ST-Link, SMPS, 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"
- note added: "Supply domain"
- note added: "USB connector"
- note added: "USB power regulator 5V to 3.3V"
- note removed: "AN3359\nst.com\n"
- note removed: "ANT\n"
- note removed: "Antenna GND"
- note removed: "Reference design from datasheet for 1.5V to 3.3V battery"
- note removed: "SMPS pravdepodobne \nnebudem vobec potrebovat"
- note removed: "Shield nechavam vysieť"
- moved on the sheet: BT1, C1, C10, C13, C17, C18, C19, C2, C3, C4, C5, C6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

Commit message: assign footprints complete need one more look and a check from Simek
Parts:
- removed J4: Conn_01x05_Male, symbol Connector:Conn_01x05_Male
- removed U3: MLL1200S TE, Package_SO:TSSOP-20_4.4x6.5mm_P0.65mm, symbol Analog_Switch:ADG734
- added J5: Conn_01x06_Male, Molexkonektor:55932-0610, symbol Connector:Conn_01x06_Male
- added S1, S2: MLL1200S, vypinac:MLL1200S, symbol BOOTSwitch:MLL1200S
- BT1: footprint Battery:BatteryHolder_Keystone_2466_1xAAA -> 0Pretty:battery_connector
- C1, C10, C13, C16, C17, C18, C19, C2, C22, C23, C24, C25, C6, C7, C8, C9, C_1: footprint (none) -> Capacitor_SMD:C_0402_1005Metric
- C11: footprint (none) -> Capacitor_SMD:C_0402_1005Metric; Buy (none) -> https://www.mouser.sk/ProductDetail/Taiyo-Yuden/LMK105BJ105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
- C12: footprint (none) -> Capacitor_SMD:C_0603_1608Metric; Buy (none) -> https://www.mouser.sk/ProductDetail/Yageo/CC0201KRX6S6BB104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
- C14: footprint (none) -> Capacitor_SMD:C_0402_1005Metric; Buy (none) -> https://www.mouser.sk/ProductDetail/Murata-Electronics/GCB1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
- C15: footprint (none) -> Capacitor_SMD:C_0402_1005Metric; Buy (none) -> https://www.mouser.sk/ProductDetail/AVX/04026D104KAT2A/?qs=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
- C20: renamed from C21; footprint (none) -> Capacitor_SMD:C_0402_1005Metric
- C21: renamed from C20; footprint (none) -> Capacitor_SMD:C_0402_1005Metric
- C3: renamed from C4; footprint (none) -> Capacitor_SMD:C_0402_1005Metric
- C4: renamed from C5; footprint (none) -> Capacitor_SMD:C_0402_1005Metric
- C5: renamed from C3; footprint (none) -> Capacitor_SMD:C_0402_1005Metric
- D1: footprint (none) -> LED_SMD:LED_0402_1005Metric
- D2: Buy (none) -> https://www.mouser.sk/ProductDetail/Vishay-Semiconductors/B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
- D3: Buy https://www.mouser.sk/ProductDetail/Diodes-Incorporated/1N4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 -> (none)
- FB1, FB2: footprint (none) -> Resistor_SMD:R_0805_2012Metric
- FB3: value MMZ2012Y152BT000 -> MMZ2012Y152BTD25; footprint (none) -> Resistor_SMD:R_0805_2012Metric
- IC1: footprint USBRegulator:SOT95P280X145-5N -> Package_TO_SOT_SMD:SOT-23-5
- IC2: footprint USB_data:SOT95P280X145-6N -> Package_TO_SOT_SMD:SOT-23-6
- J2: footprint (none) -> Molexkonektor:55932-0610
- J3: renamed from J5; footprint (none) -> 0Pretty:PCB_Pin_connector
- J4: renamed from J3; footprint (none) -> 0Pretty:Pin_FSR
- L1, L3: footprint (none) -> Inductor_SMD:L_0603_1608Metric
- L2: footprint (none) -> 0Pretty:L_0712_SMD
- R1, R10, R11, R12, R13, R2, R3, R4, R5, R6, R7, R8, R9, R_1, R_2: footprint (none) -> Resistor_SMD:R_0402_1005Metric
- U2: Buy (none) -> https://www.mouser.sk/ProductDetail/STMicroelectronics/STM3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
- U4: Buy (none) -> https://www.mouser.sk/ProductDetail/Bosch-Sensortec/BNO055/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
- U5: footprint Package_SO:TSSOP-10_3x3mm_P0.5mm -> ADS1115:ADS1115IRUGR
- Y2, Y3: footprint Crystal:Crystal_SMD_2012-2Pin_2.0x1.2mm -> 0Pretty:Crystal_2012_custom
Connections:
- net +3V3: now also J5.1 (Pin_1), S1.1 (NC), S2.2 (COM)
- net 3v3fromBAT: now also S2.1 (NC)
- net 3v3fromUSB: now also S2.3 (NO)
- net GND: now also J5.6 (Pin_6)
- net NRST: now also J5.2 (Pin_2)
- net SYS_JTCK-SWCLK: now also J5.4 (Pin_4)
- net SYS_JTDO-SWO: now also J5.5 (Pin_5)
- net SYS_JTMS-SWDIO: now also J5.3 (Pin_3)
- net at R4.1, U2.4 (PH3-BOOT0): now also S1.2 (COM)
- no-connect marks 17 -> 23
Other:
- note added: "Boot mode selection switch\nBOOT=0 Default position, connected to GND\nBOOT=1 Connected to 3.3V"
- note removed: "BOOT=0 Default position, connected to GND\nBOOT=1 Connected to 3.3V"
- moved on the sheet: C17, C18, C19, C21, C23, C24, C25, C5, D1, D2, FB1, J3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

Commit message: dokoncene rozlozenie okolo STM32WB podla referencneho dizajnu
Parts:
- removed J3: Conn_01x03_Male, 0Pretty:PCB_Pin_connector, symbol Connector:Conn_01x03_Male
- removed J5: Conn_01x06_Male, Molexkonektor:55932-0610, symbol Connector:Conn_01x06_Male
- removed R10, R11: 10K, Resistor_SMD:R_0402_1005Metric, symbol Device:R_Small
- removed Y1: NX2520SA-32MHz, Crystal:Crystal_SMD_2520-4Pin_2.5x2.0mm, symbol Device:Crystal_GND3_Small
- added C26, C27: 100n, Capacitor_SMD:C_0402_1005Metric, symbol Device:C_Small
- added J3: Conn_01x02_Male, 0Pretty:pin_02, symbol Connector:Conn_01x02_Male
- added J5, J6: Conn_01x01_Male, 0Pretty:pin_01, symbol Connector:Conn_01x01_Male
- added J7: Conn_01x08_Male, 0Pretty:pin_08, symbol Connector:Conn_01x08_Male
- added Y1: NX2520SA-32MHz, Crystal:Crystal_SMD_2520-4Pin_2.5x2.0mm, symbol USB_svab:Crystal_GND3_Small
- BT1: footprint 0Pretty:battery_connector -> 0Pretty:battery_connector_narrow
- C23: value 1u -> 100n
- D1: footprint LED_SMD:LED_0402_1005Metric -> LED_SMD:LED_0603_1608Metric
- FB1: value Z0805C601BSMST -> BLM15AX601SN1D; footprint Resistor_SMD:R_0805_2012Metric -> Resistor_SMD:R_0402_1005Metric
- FB2, FB3: footprint Resistor_SMD:R_0805_2012Metric -> Resistor_SMD:R_0402_1005Metric
- J2: value Conn_01x06_Male -> Conn_01x05_Male; footprint Molexkonektor:55932-0610 -> 0Pretty:pin_03; symbol Connector:Conn_01x06_Male -> Connector:Conn_01x03_Male
Connections:
- net +3V3: now also U4.28 (VDDIO), U4.3 (VDD), C26.1, C27.1, J7.1 (Pin_1)
- net BNO055_RESET: now also J5.1 (Pin_1); no longer J2.4 (Pin_4)
- net GENERAL_PIN_OUT1: now also U2.42 (PA15), J7.4 (Pin_4); no longer U2.14 (PA5)
- net GENERAL_PIN_OUT2: now also J7.6 (Pin_6)
- net GENERAL_PIN_OUT3: now also J7.7 (Pin_7)
- net GND: now also U4.10 (BL_IND), U4.2 (GND), U4.5 (PS1), U4.6 (PS0), C26.2, C27.2, J7.8 (Pin_8), Y1.2, Y1.4; no longer U4.28 (VDDIO)
- net I2C_SCL: now also J3.1 (Pin_1); no longer J2.5 (Pin_5)
- net I2C_SDA: now also J3.2 (Pin_2); no longer J2.6 (Pin_6)
- net NRST: now also J6.1 (Pin_1)
- net SYS_JTCK-SWCLK: now also J7.3 (Pin_3)
- net SYS_JTDO-SWO: now also J7.5 (Pin_5)
- net SYS_JTMS-SWDIO: now also J7.2 (Pin_2)
- net at U2.24 (OSC_OUT/RCC_OSC_OUT): now also Y1.1
- net at U2.25 (OSC_IN/RCC_OSC_IN): now also Y1.3
- net USB_OD+: now reaches IC2.4 (USB_O_D+), J1.3 (D+)
- net USB_OD-: now reaches IC2.6 (USB_O_D-), J1.2 (D-)
- net at U4.27 (XIN32): now also C25.1, Y3.2
Other:
- note added: "ADDR \n0x28 GND\n0x29 NC"
- moved on the sheet: C20, C21, C22, C23, C24, C25, D3, FB2, FB3, J4, R12, R13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
